File: pcb/Y8960_Cartridge/Y8960_Cartridge.kicad_sch (KiCad schematic)
At the start: 58 parts, among them J1 I2S_CONN, J2 SOUNDIN, J3 Conn_02x06_Odd_Even, J4 GND, Q1 NMOS, Q2 NMOS, Q3 NMOS

Commit message: Updated
Parts:
- C4: footprint Capacitor_THT:CP_Radial_D5.0mm_P2.50mm -> Capacitor_SMD:C_1210_3225Metric_Pad1.33x2.70mm_HandSolder
Changed lines of the file:
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@@
 			)
 		)
-		(property "Footprint" "Capacitor_THT:CP_Radial_D5.0mm_P2.50mm"
+		(property "Footprint" "Capacitor_SMD:C_1210_3225Metric_Pad1.33x2.70mm_HandSolder"
 			(at 166.0652 273.05 0)
 			(effects

Commit message: Updated
Parts:
- C1, C10, C11, C12, C3, C5, C6, C7, C8, C9: footprint Capacitor_SMD:C_0805_2012Metric_Pad1.18x1.45mm_HandSolder -> Capacitor_SMD:C_0402_1005Metric; LCSC (none) -> C1525
- C2: footprint Capacitor_SMD:C_0805_2012Metric_Pad1.18x1.45mm_HandSolder -> Capacitor_SMD:C_0805_2012Metric; LCSC (none) -> C63339
- C4: footprint Capacitor_SMD:C_1210_3225Metric_Pad1.33x2.70mm_HandSolder -> Capacitor_SMD:C_1210_3225Metric; LCSC (none) -> C49066
- D1, D2, D3, D4: footprint LED_SMD:LED_0805_2012Metric_Pad1.15x1.40mm_HandSolder -> LED_SMD:LED_0805_2012Metric; LCSC (none) -> C84256
- Q1, Q2, Q3: LCSC (none) -> C458143
- R1, R13, R14, R15, R16, R17, R18, R2, R3, R4, R5, R6, R7, R8: footprint Resistor_SMD:R_0805_2012Metric_Pad1.20x1.40mm_HandSolder -> Resistor_SMD:R_0805_2012Metric; LCSC (none) -> C104350
- R10, R11, R12, R19, R21, R9: footprint Resistor_SMD:R_0805_2012Metric_Pad1.20x1.40mm_HandSolder -> Resistor_SMD:R_0805_2012Metric; LCSC (none) -> C26010
- R20: footprint Resistor_SMD:R_0805_2012Metric_Pad1.20x1.40mm_HandSolder -> Resistor_SMD:R_0805_2012Metric; LCSC (none) -> C17414
- R24, R25, R26, R27: footprint Resistor_SMD:R_0805_2012Metric_Pad1.20x1.40mm_HandSolder -> Resistor_SMD:R_0805_2012Metric; LCSC (none) -> C17710
- U1: LCSC (none) -> C597938; note (none) -> Use two specified connectors
- U2: note (none) -> Card edge
- U3: LCSC (none) -> C387408
- U4, U5, U6, U7: LCSC (none) -> C19197
- U8: LCSC (none) -> C27585175

Commit message: Updated
Parts:
- removed U1: ~, 0-My_Parts:TangPrimer25K, symbol My_Symbols:Y8960
- added U1: ~, 0-My_Parts:TangPrimer25K(UPPER), symbol My_Symbols:Y8960(UPPER)
- added U9: ~, 0-My_Parts:TangPrimer25K(LOWER), symbol My_Symbols:Y8960(LOWER)
Connections:
- net +3V3: now also U1.2 (VCCIO2/3), U1.4 (VCCIO2/3), U1.46 (VDD_3V3), U1.48 (VDD_3V3), U1.50 (VDD_3V3), U9.84 (VCCIO0/1), U9.86 (VCCIO0/1), U9.89 (VCCIO6/7), U9.91 (VCCIO6/7)
- net +5V: now also U1.52 (VDD_5V), U1.54 (VDD_5V), U1.56 (VDD_5V), U1.58 (VDD_5V), U1.60 (VDD_5V)
- net AUDIO_BCLK: now also U9.114 (AUDIO_BCLK)
- net AUDIO_LRCLK: now also U9.116 (AUDIO_LRCLK)
- net AUDIO_MCLK: now also U9.112 (AUDIO_MCLK)
- net AUDIO_SDATA: now also U9.118 (AUDIO_SDATA)
- net CLK28M: now also U9.64 (CLK28M)
- net DIPSW0: now also U9.77 (DIPSW0(READY))
- net DIPSW1: now also U9.83 (DIPSW1)
- net GND: now also U1.1 (GND), U1.19 (GND), U1.29 (GND), U1.35 (GND), U1.41 (GND), U1.47 (GND), U1.53 (GND), U1.59 (GND), U9.105 (GND), U9.110 (GND), U9.119 (GND), U9.120 (GND), U9.61 (GND), U9.62 (GND), U9.75 (GND), U9.87 (GND), U9.88 (GND)
- net JTAG_TCK: now also U1.21 (JTAG_TCK)
- net JTAG_TDI: now also U1.27 (JTAG_TDI)
- net JTAG_TDO: now also U1.25 (JTAG_TDO)
- net JTAG_TMS: now also U1.23 (JTAG_TMS)
- net SLOT_A0: now also U9.63 (SLOT_A0)
- net SLOT_A1: now also U9.65 (SLOT_A1)
- net SLOT_A10: now also U9.78 (SLOT_A10)
- net SLOT_A11: now also U9.76 (SLOT_A11)
- net SLOT_A12: now also U9.74 (SLOT_A12)
- net SLOT_A13: now also U9.72 (SLOT_A13)
- net SLOT_A14: now also U9.108 (SLOT_A14)
- net SLOT_A15: now also U9.106 (SLOT_A15)
- net SLOT_A2: now also U9.67 (SLOT_A2)
- net SLOT_A3: now also U9.69 (SLOT_A3)
- net SLOT_A4: now also U9.71 (SLOT_A4)
- net SLOT_A5: now also U9.73 (SLOT_A5)
- net SLOT_A6: now also U9.93 (SLOT_A6)
- net SLOT_A7: now also U9.95 (SLOT_A7)
- net SLOT_A8: now also U9.82 (SLOT_A8)
- net SLOT_A9: now also U9.80 (SLOT_A9)
- net SLOT_BUSDIR: now also U9.103 (SLOT_BUSDIR)
- net SLOT_D0: now also U9.90 (SLOT_D0)
- net SLOT_D1: now also U9.92 (SLOT_D1)
- net SLOT_D2: now also U9.94 (SLOT_D2)
- net SLOT_D3: now also U9.96 (SLOT_D3)
- net SLOT_D4: now also U9.98 (SLOT_D4)
- net SLOT_D5: now also U9.100 (SLOT_D5)
- net SLOT_D6: now also U9.102 (SLOT_D6)
- net SLOT_D7: now also U9.104 (SLOT_D7)
- net SLOT_INTR: now also U9.97 (SLOT_INTR)
- net SLOT_IORQ_N: now also U9.68 (SLOT_IORQ_N)
- net SLOT_M1_N: now also U1.6 (SLOT_M1_N)
- net SLOT_MERQ_N: now also U9.70 (SLOT_MERQ_N)
- net SLOT_RD_N: now also U9.109 (SLOT_RD_N)
- net SLOT_RESET_N: now also U9.101 (SLOT_RESET_N)
- net SLOT_SLTSL_N: now also U9.66 (SLOT_SLTSL_N)
- net SLOT_WAIT: now also U9.99 (SLOT_WAIT)
- net SLOT_WR_N: now also U9.107 (SLOT_WR_N)
- net SRAM_CS_N: now also U1.9 (SRAM_CS_N)
- net SRAM_SCLK: now also U1.7 (SRAM_SCLK)
- net SRAM_SIO0: now also U1.11 (SRAM_SIO0)
- net SRAM_SIO1: now also U1.5 (SRAM_SIO1)
- net SRAM_SIO2: now also U1.15 (SRAM_SIO2)
- net SRAM_SIO3: now also U1.17 (SRAM_SIO3)
- net UART_RX: now also U9.79 (UART_RX)
- net UART_TX: now also U9.81 (UART_TX)
- net at D1.1 (K): now also U9.111 (LED0)
- net at D2.1 (K): now also U9.113 (LED1)
- net at D4.1 (K): now also U9.117 (LED3)
- net at D3.1 (K): now also U9.115 (LED2)
