File: pcb/Y8960_Cartridge/Y8960_Cartridge.kicad_pcb (KiCad board)
At the start: 2 copper layers, 95.2 x 65.4 mm, 60 parts, among them J1 I2S_CONN, J2 SOUNDIN, J3 Conn_02x06_Odd_Even, J4 GND, Q1 NMOS, Q2 NMOS, Q3 NMOS

Commit message: Updated
Parts:
- C4: footprint Capacitor_THT:CP_Radial_D5.0mm_P2.50mm -> Capacitor_SMD:C_1210_3225Metric_Pad1.33x2.70mm_HandSolder
- moved C4 1.71 mm to (72.8, 102.4)
Routing:
- net GND: track 404.7 -> 404.0 mm
- net +5V: vias 7 -> 8

Commit message: Updated
Parts:
- C1, C10, C11, C12, C3, C5, C6, C7, C8, C9: footprint Capacitor_SMD:C_0805_2012Metric_Pad1.18x1.45mm_HandSolder -> Capacitor_SMD:C_0402_1005Metric
- C2: footprint Capacitor_SMD:C_0805_2012Metric_Pad1.18x1.45mm_HandSolder -> Capacitor_SMD:C_0805_2012Metric
- C4: footprint Capacitor_SMD:C_1210_3225Metric_Pad1.33x2.70mm_HandSolder -> Capacitor_SMD:C_1210_3225Metric
- D1, D2, D3, D4: footprint LED_SMD:LED_0805_2012Metric_Pad1.15x1.40mm_HandSolder -> LED_SMD:LED_0805_2012Metric
- R1, R10, R11, R12, R13, R14, R15, R16, R17, R18, R19, R2, R20, R21, R24, R25, R26, R27, R3, R4, R5, R6, R7, R8, R9: footprint Resistor_SMD:R_0805_2012Metric_Pad1.20x1.40mm_HandSolder -> Resistor_SMD:R_0805_2012Metric
- moved C2 2.18 mm to (91.4, 71.5)
Routing:
- net GND: track 404.0 -> 415.5 mm, vias 105 -> 117
- net +3V3: track 298.5 -> 302.4 mm
- net +5V: track 213.2 -> 215.3 mm
- net CLK28M: track 19.4 -> 20.9 mm

Commit message: Updated
Parts:
- added U9: ~, 0-My_Parts:TangPrimer25K(LOWER), F.Cu at (114.8, 79.3)
- U1: footprint 0-My_Parts:TangPrimer25K -> 0-My_Parts:TangPrimer25K(UPPER)
Other:
- board text added: "TangPrimer25K"

Commit message: Updated
Other:
- board text added: "OFF"
- board text added: "ON"
- board text added: "ROM"
Changed lines of the file:
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@@
+		)
+	)
+	(gr_text "ROM"
+		(at 99.025 70.4 0)
+		(layer "F.SilkS")
+		(effects
+			(font
+				(size 1 1)
+				(thickness 0.1)
+			)
+			(justify left bottom)
 		)
 	)
@@
 	(gr_text "DI"
 		(at 152.95 79.875 0)
+		(layer "F.SilkS")
+		(effects
+			(font
+				(size 1 1)
+				(thickness 0.1)
+			)
+			(justify left bottom)
+		)
+	)
+	(gr_text "OFF"
+		(at 99.225 72.6 0)
 		(layer "F.SilkS")
 		(effects
@@
 		)
 	)
+	(gr_text "ON"
+		(at 99.575 77.75 0)
+		(layer "F.SilkS")
+		(effects
+			(font
+				(size 1 1)
+				(thickness 0.1)
+			)
+			(justify left bottom)
+		)
+	)
